Commit message: Revert "[data] Fix mesh paths to match franka_description"
This reverts commit c7792ffedd7d059e3fb01e4ef5a20dd5c8ea8a9a.

File: data/xacro/hand.xacro (robot description, xacro)
@@ -20,5 +20,5 @@
       <visual>
         <geometry>
-          <mesh filename="package://franka_description/meshes/robot_ee/franka_hand_white/visual/hand.dae"/>
+          <mesh filename="package://franka_description/meshes/visual/hand.dae"/>
         </geometry>
       </visual>
@@ -63,5 +63,5 @@
       <visual>
         <geometry>
-          <mesh filename="package://franka_description/meshes/robot_ee/franka_hand_white/visual/finger.dae"/>
+          <mesh filename="package://franka_description/meshes/visual/finger.dae"/>
         </geometry>
       </visual>
@@ -71,5 +71,5 @@
         <origin xyz="0 0 0" rpy="0 0 ${pi}"/>
         <geometry>
-          <mesh filename="package://franka_description/meshes/robot_ee/franka_hand_white/visual/finger.dae"/>
+          <mesh filename="package://franka_description/meshes/visual/finger.dae"/>
         </geometry>
       </visual>
