Commit message: Fix URDF generation without ROS

File: data/urdf/panda_default.urdf (robot description, URDF)
Before this commit: robot panda_default, 11 links, 10 joints
Links:
- link panda_link0: geometry collision cylinder length=0.03 radius=0.09; collision sphere radius=0.09
- link panda_link1: geometry collision cylinder length=0.2830 radius=0.09; collision sphere radius=0.09
- link panda_link2: geometry collision cylinder length=0.12 radius=0.09; collision sphere radius=0.09
- link panda_link3: geometry collision cylinder length=0.15 radius=0.09; collision sphere radius=0.09
- link panda_link4: geometry collision cylinder length=0.12 radius=0.09; collision sphere radius=0.09
- link panda_link5: geometry collision cylinder length=0.1 radius=0.09; collision cylinder length=0.14 radius=0.055
- link panda_link6: geometry collision cylinder length=0.08 radius=0.08; collision sphere radius=0.08
- link panda_link7: geometry collision cylinder length=0.14 radius=0.07; collision sphere radius=0.07

File: data/urdf/panda_foot.urdf (robot description, URDF)
Before this commit: robot panda_foot, 12 links, 11 joints
Links:
- link panda_foot: geometry collision mesh filename=file://@URDF_DESTINATION@/meshes/foot.stl; visual mesh filename=file://@URDF_DESTINATION@/meshes/foot.stl
- link panda_link0: geometry collision cylinder length=0.03 radius=0.09; collision sphere radius=0.09
- link panda_link1: geometry collision cylinder length=0.2830 radius=0.09; collision sphere radius=0.09
- link panda_link2: geometry collision cylinder length=0.12 radius=0.09; collision sphere radius=0.09
- link panda_link3: geometry collision cylinder length=0.15 radius=0.09; collision sphere radius=0.09
- link panda_link4: geometry collision cylinder length=0.12 radius=0.09; collision sphere radius=0.09
- link panda_link5: geometry collision cylinder length=0.1 radius=0.09; collision cylinder length=0.14 radius=0.055
- link panda_link6: geometry collision cylinder length=0.08 radius=0.08; collision sphere radius=0.08
- link panda_link7: geometry collision cylinder length=0.14 radius=0.07; collision sphere radius=0.07

File: data/urdf/panda_hand.urdf (robot description, URDF)
Before this commit: robot panda_hand, 14 links, 13 joints
Links:
- link panda_hand: geometry collision cylinder length=0.1 radius=0.02; collision cylinder length=0.1 radius=0.04
- link panda_leftfinger: geometry visual mesh filename=file://@URDF_DESTINATION@/meshes/visual/finger.dae
- link panda_link0: geometry collision cylinder length=0.03 radius=0.09; collision sphere radius=0.09
- link panda_link1: geometry collision cylinder length=0.2830 radius=0.09; collision sphere radius=0.09
- link panda_link2: geometry collision cylinder length=0.12 radius=0.09; collision sphere radius=0.09
- link panda_link3: geometry collision cylinder length=0.15 radius=0.09; collision sphere radius=0.09
- link panda_link4: geometry collision cylinder length=0.12 radius=0.09; collision sphere radius=0.09
- link panda_link5: geometry collision cylinder length=0.1 radius=0.09; collision cylinder length=0.14 radius=0.055
- link panda_link6: geometry collision cylinder length=0.08 radius=0.08; collision sphere radius=0.08
- link panda_link7: geometry collision cylinder length=0.14 radius=0.07; collision sphere radius=0.07
- link panda_rightfinger: geometry visual mesh filename=file://@URDF_DESTINATION@/meshes/visual/finger.dae

File: data/urdf/panda_pump.urdf (robot description, URDF)
Before this commit: robot panda_pump, 12 links, 11 joints
Links:
- link panda_link0: geometry collision cylinder length=0.03 radius=0.09; collision sphere radius=0.09
- link panda_link1: geometry collision cylinder length=0.2830 radius=0.09; collision sphere radius=0.09
- link panda_link2: geometry collision cylinder length=0.12 radius=0.09; collision sphere radius=0.09
- link panda_link3: geometry collision cylinder length=0.15 radius=0.09; collision sphere radius=0.09
- link panda_link4: geometry collision cylinder length=0.12 radius=0.09; collision sphere radius=0.09
- link panda_link5: geometry collision cylinder length=0.1 radius=0.09; collision cylinder length=0.14 radius=0.055
- link panda_link6: geometry collision cylinder length=0.08 radius=0.08; collision sphere radius=0.08
- link panda_link7: geometry collision cylinder length=0.14 radius=0.07; collision sphere radius=0.07
- link panda_pump: geometry collision mesh filename=file://@URDF_DESTINATION@/meshes/pump.dae; visual mesh filename=file://@URDF_DESTINATION@/meshes/pump.dae

Commit message: Use the inertial parameters released by Franka Emika

File: data/urdf/panda_default.urdf (robot description, URDF)
Before this commit: robot panda_default, 11 links, 10 joints
Links:
- link panda_link0: mass 2.92 -> 0.629769
- link panda_link1: mass 2.74 -> 4.970684
- link panda_link2: mass 2.74 -> 0.646926
- link panda_link3: mass 2.38 -> 3.228604
- link panda_link4: mass 2.38 -> 3.587895
- link panda_link5: mass 2.74 -> 1.225946
- link panda_link6: mass 1.55 -> 1.666555
- link panda_link7: mass 0.54 -> 7.35522e-01
Joints:
- joint panda_joint2: origin xyz=0 0 0 rpy=-1.57079632679 0 0 -> xyz=0 0 0 rpy=-1.5707963267948966 0 0
- joint panda_joint3: origin xyz=0 -0.316 0 rpy=1.57079632679 0 0 -> xyz=0 -0.316 0 rpy=1.5707963267948966 0 0
- joint panda_joint4: origin xyz=0.0825 0 0 rpy=1.57079632679 0 0 -> xyz=0.0825 0 0 rpy=1.5707963267948966 0 0
- joint panda_joint5: origin xyz=-0.0825 0.384 0 rpy=-1.57079632679 0 0 -> xyz=-0.0825 0.384 0 rpy=-1.5707963267948966 0 0
- joint panda_joint6: origin xyz=0 0 0 rpy=1.57079632679 0 0 -> xyz=0 0 0 rpy=1.5707963267948966 0 0
- joint panda_joint7: origin xyz=0.088 0 0 rpy=1.57079632679 0 0 -> xyz=0.088 0 0 rpy=1.5707963267948966 0 0

File: data/urdf/panda_foot.urdf (robot description, URDF)
Before this commit: robot panda_foot, 12 links, 11 joints
Links:
- link panda_link0: mass 2.92 -> 0.629769
- link panda_link1: mass 2.74 -> 4.970684
- link panda_link2: mass 2.74 -> 0.646926
- link panda_link3: mass 2.38 -> 3.228604
- link panda_link4: mass 2.38 -> 3.587895
- link panda_link5: mass 2.74 -> 1.225946
- link panda_link6: mass 1.55 -> 1.666555
- link panda_link7: mass 0.54 -> 7.35522e-01
Joints:
- joint panda_foot_joint: origin xyz=0 0 0 rpy=0 0 -0.785398163397 -> xyz=0 0 0 rpy=0 0 -0.7853981633974483
- joint panda_joint2: origin xyz=0 0 0 rpy=-1.57079632679 0 0 -> xyz=0 0 0 rpy=-1.5707963267948966 0 0
- joint panda_joint3: origin xyz=0 -0.316 0 rpy=1.57079632679 0 0 -> xyz=0 -0.316 0 rpy=1.5707963267948966 0 0
- joint panda_joint4: origin xyz=0.0825 0 0 rpy=1.57079632679 0 0 -> xyz=0.0825 0 0 rpy=1.5707963267948966 0 0
- joint panda_joint5: origin xyz=-0.0825 0.384 0 rpy=-1.57079632679 0 0 -> xyz=-0.0825 0.384 0 rpy=-1.5707963267948966 0 0
- joint panda_joint6: origin xyz=0 0 0 rpy=1.57079632679 0 0 -> xyz=0 0 0 rpy=1.5707963267948966 0 0
- joint panda_joint7: origin xyz=0.088 0 0 rpy=1.57079632679 0 0 -> xyz=0.088 0 0 rpy=1.5707963267948966 0 0

File: data/urdf/panda_hand.urdf (robot description, URDF)
Before this commit: robot panda_hand, 14 links, 13 joints
Links:
- link panda_hand: mass None -> 0.73
- link panda_link0: mass 2.92 -> 0.629769
- link panda_link1: mass 2.74 -> 4.970684
- link panda_link2: mass 2.74 -> 0.646926
- link panda_link3: mass 2.38 -> 3.228604
- link panda_link4: mass 2.38 -> 3.587895
- link panda_link5: mass 2.74 -> 1.225946
- link panda_link6: mass 1.55 -> 1.666555
- link panda_link7: mass 0.54 -> 7.35522e-01
Joints:
- joint panda_hand_joint: origin xyz=0 0 0 rpy=0 0 -0.785398163397 -> xyz=0 0 0 rpy=0 0 -0.7853981633974483
- joint panda_joint2: origin xyz=0 0 0 rpy=-1.57079632679 0 0 -> xyz=0 0 0 rpy=-1.5707963267948966 0 0
- joint panda_joint3: origin xyz=0 -0.316 0 rpy=1.57079632679 0 0 -> xyz=0 -0.316 0 rpy=1.5707963267948966 0 0
- joint panda_joint4: origin xyz=0.0825 0 0 rpy=1.57079632679 0 0 -> xyz=0.0825 0 0 rpy=1.5707963267948966 0 0
- joint panda_joint5: origin xyz=-0.0825 0.384 0 rpy=-1.57079632679 0 0 -> xyz=-0.0825 0.384 0 rpy=-1.5707963267948966 0 0
- joint panda_joint6: origin xyz=0 0 0 rpy=1.57079632679 0 0 -> xyz=0 0 0 rpy=1.5707963267948966 0 0
- joint panda_joint7: origin xyz=0.088 0 0 rpy=1.57079632679 0 0 -> xyz=0.088 0 0 rpy=1.5707963267948966 0 0

File: data/urdf/panda_pump.urdf (robot description, URDF)
Before this commit: robot panda_pump, 12 links, 11 joints
Links:
- link panda_link0: mass 2.92 -> 0.629769
- link panda_link1: mass 2.74 -> 4.970684
- link panda_link2: mass 2.74 -> 0.646926
- link panda_link3: mass 2.38 -> 3.228604
- link panda_link4: mass 2.38 -> 3.587895
- link panda_link5: mass 2.74 -> 1.225946
- link panda_link6: mass 1.55 -> 1.666555
- link panda_link7: mass 0.54 -> 7.35522e-01
Joints:
- joint panda_joint2: origin xyz=0 0 0 rpy=-1.57079632679 0 0 -> xyz=0 0 0 rpy=-1.5707963267948966 0 0
- joint panda_joint3: origin xyz=0 -0.316 0 rpy=1.57079632679 0 0 -> xyz=0 -0.316 0 rpy=1.5707963267948966 0 0
- joint panda_joint4: origin xyz=0.0825 0 0 rpy=1.57079632679 0 0 -> xyz=0.0825 0 0 rpy=1.5707963267948966 0 0
- joint panda_joint5: origin xyz=-0.0825 0.384 0 rpy=-1.57079632679 0 0 -> xyz=-0.0825 0.384 0 rpy=-1.5707963267948966 0 0
- joint panda_joint6: origin xyz=0 0 0 rpy=1.57079632679 0 0 -> xyz=0 0 0 rpy=1.5707963267948966 0 0
- joint panda_joint7: origin xyz=0.088 0 0 rpy=1.57079632679 0 0 -> xyz=0.088 0 0 rpy=1.5707963267948966 0 0
- joint panda_pump_joint: origin xyz=0 0 0 rpy=0 0 -0.785398163397 -> xyz=0 0 0 rpy=0 0 -0.7853981633974483

File: data/xacro/hand.xacro (robot description, xacro)
@@ -11,4 +11,11 @@
     </xacro:unless>
     <link name="${ns}_hand">
+      <inertial>
+        <mass value="0.73" />
+        <origin xyz="-0.01 0 0.03" />
+        <inertia ixx="0.001" ixy="0"      ixz="0"
+                             iyy="0.0025" iyz="0"
+                                          izz="0.0017" />
+      </inertial>
       <visual>
         <geometry>

File: data/xacro/panda.xacro (robot description, xacro)
@@ -19,7 +19,10 @@
     <link name="${arm_id}_link0">
       <inertial>
-        <mass value="2.92" />
-        <origin xyz="-0.025566 -2.88e-05 0.057332" rpy="0 0 0" />
-        <inertia ixx="0.00782229414331" ixy="-1.56191622996e-05" ixz="-0.00126005738123" iyy="0.0109027971813" iyz="1.08233858202e-05" izz="0.0102355503949" />
+        <!-- Estimated guesses from CAD -->
+        <origin rpy="0 0 0" xyz="-0.041018 -0.00014 0.049974"/>
+        <mass value="0.629769"/>
+        <inertia ixx="0.00315" ixy="8.2904E-07" ixz="0.00015"
+                               iyy="0.00388"    iyz="8.2299E-06"
+                                                izz="0.004285" />
       </inertial>
       <visual>
@@ -53,7 +56,9 @@
     <link name="${arm_id}_link1">
       <inertial>
-        <mass value="2.74" />
-        <origin xyz="0 -0.0324958 -0.0675818" rpy="0 0 0" />
-        <inertia ixx="0.0180416958283" ixy="0.0" ixz="0.0" iyy="0.0159136071891" iyz="0.0046758424612" izz="0.00620690827127" />
+        <origin rpy="0 0 0" xyz="0.003875 0.002081 -0.04762"/>
+        <mass value="4.970684"/>
+        <inertia ixx="0.70337" ixy="-0.00013900" ixz="0.0067720"
+                               iyy="0.70661"     iyz="0.019169"
+                                                 izz="0.0091170" />
       </inertial>
       <visual>
@@ -95,7 +100,9 @@
     <link name="${arm_id}_link2">
       <inertial>
-        <mass value="2.74" />
-        <origin xyz="0 -0.06861 0.0322285" rpy="0 0 0" />
-        <inertia ixx="0.0182856182281" ixy="0.0" ixz="0.0" iyy="0.00621358421175" iyz="-0.00472844221905" izz="0.0161514346309" />
+        <origin rpy="0 0 0" xyz=" -0.003141 -0.02872  0.003495"/>
+        <mass value="0.646926"/>
+        <inertia ixx="0.0079620" ixy="-3.9250e-3" ixz="1.0254e-02"
+                                 iyy="2.8110e-02" iyz="7.0400e-04"
+                                                  izz="2.5995e-02" />
       </inertial>
       <visual>
@@ -137,7 +144,9 @@
     <link name="${arm_id}_link3">
       <inertial>
-        <mass value="2.38" />
-        <origin xyz="0.0469893 0.0316374 -0.031704" rpy="0 0 0" />
-        <inertia ixx="0.00771376630908" ixy="-0.00248490625138" ixz="-0.00332147581033" iyy="0.00989108008727" iyz="-0.00217796151484" izz="0.00811723558464" />
+        <origin rpy="0 0 0" xyz="2.7518e-02 3.9252e-02 -6.6502e-02"/>
+        <mass value="3.228604"/>
+        <inertia ixx="3.7242e-02" ixy="-4.7610e-03" ixz="-1.1396e-02"
+                                  iyy="3.6155e-02"  iyz="-1.2805e-02"
+                                                    izz="1.0830e-02" />
       </inertial>
       <visual>
@@ -179,7 +188,9 @@
     <link name="${arm_id}_link4">
       <inertial>
-        <mass value="2.38" />
-        <origin xyz="-0.0360446 0.0336853 0.031882" rpy="0 0 0" />
-        <inertia ixx="0.00799663881132" ixy="0.00347095570217" ixz="-0.00241222942995" iyy="0.00825390705278" iyz="0.00235774044121" izz="0.0102515004345" />
+        <origin rpy="0 0 0" xyz="-5.317e-02 1.04419e-01 2.7454e-02"/>
+        <mass value="3.587895"/>
+        <inertia ixx="2.5853e-02" ixy="7.7960e-03" ixz="-1.3320e-03"
+                                  iyy="1.9552e-02" iyz="8.6410e-03"
+                                                   izz="2.8323e-02" />
       </inertial>
       <visual>
@@ -221,7 +232,9 @@
     <link name="${arm_id}_link5">
       <inertial>
-        <mass value="2.74" />
-        <origin xyz="0 0.0610427 -0.104176" rpy="0 0 0" />
-        <inertia ixx="0.030371374513" ixy="6.50283587108e-07" ixz="-1.05129179916e-05" iyy="0.0288752887402" iyz="-0.00775653445787" izz="0.00444134056164" />
+        <origin rpy="0 0 0" xyz="-1.1953e-02 4.1065e-02 -3.8437e-02"/>
+        <mass value="1.225946"/>
+        <inertia ixx="3.5549e-02" ixy="-2.1170e-03" ixz="-4.0370e-03"
+                                  iyy="2.9474e-02"  iyz="2.2900e-04"
+                                                    izz="8.6270e-03" />
       </inertial>
       <visual>
@@ -281,7 +294,9 @@
     <link name="${arm_id}_link6">
       <inertial>
-        <mass value="1.55" />
-        <origin xyz="0.0510509 0.009108 0.0106343" rpy="0 0 0" />
-        <inertia ixx="0.00303336450376" ixy="-0.000437276865508" ixz="0.000629257294877" iyy="0.00404479911567" iyz="0.000130472021025" izz="0.00558234286039" />
+        <origin rpy="0 0 0" xyz="6.0149e-02 -1.4117e-02 -1.0517e-02"/>
+        <mass value="1.666555"/>
+        <inertia ixx="1.9640e-03" ixy="1.0900e-04" ixz="-1.1580e-03"
+                                  iyy="4.3540e-03" iyz="3.4100e-04"
+                                                   izz="5.4330e-03" />
       </inertial>
       <visual>
@@ -323,7 +338,9 @@
     <link name="${arm_id}_link7">
       <inertial>
-        <mass value="0.54" />
-        <origin xyz="0.0109695 0.0107965 0.0650411" rpy="0 0 0" />
-        <inertia ixx="0.000888868887021" ixy="-0.00012239074652" ixz="3.98699829666e-05" iyy="0.000888001373233" iyz="-9.33825115206e-05" izz="0.0007176834609" />
+        <origin rpy="0 0 0" xyz="1.0517e-02 -4.252e-03 6.1597e-02"/>
+        <mass value="7.35522e-01"/>
+        <inertia ixx="1.2516e-02" ixy="-4.2800e-04" ixz="-1.1960e-03"
+                                  iyy="1.0027e-02"  iyz="-7.4100e-04"
+                                                    izz="4.8150e-03"/>
       </inertial>
       <visual>

Commit message: [data] Fix mesh paths to match franka_description

File: data/urdf/panda_default.urdf (robot description, URDF)
Before this commit: robot panda_default, 11 links, 10 joints
Links:
- link panda_link0: geometry collision cylinder length=0.03 radius=0.09; collision sphere radius=0.09
- link panda_link1: geometry collision cylinder length=0.2830 radius=0.09; collision sphere radius=0.09
- link panda_link2: geometry collision cylinder length=0.12 radius=0.09; collision sphere radius=0.09
- link panda_link3: geometry collision cylinder length=0.15 radius=0.09; collision sphere radius=0.09
- link panda_link4: geometry collision cylinder length=0.12 radius=0.09; collision sphere radius=0.09
- link panda_link5: geometry collision cylinder length=0.1 radius=0.09; collision cylinder length=0.14 radius=0.055
- link panda_link6: geometry collision cylinder length=0.08 radius=0.08; collision sphere radius=0.08
- link panda_link7: geometry collision cylinder length=0.14 radius=0.07; collision sphere radius=0.07

File: data/urdf/panda_foot.urdf (robot description, URDF)
Before this commit: robot panda_foot, 12 links, 11 joints
Links:
- link panda_link0: geometry collision cylinder length=0.03 radius=0.09; collision sphere radius=0.09
- link panda_link1: geometry collision cylinder length=0.2830 radius=0.09; collision sphere radius=0.09
- link panda_link2: geometry collision cylinder length=0.12 radius=0.09; collision sphere radius=0.09
- link panda_link3: geometry collision cylinder length=0.15 radius=0.09; collision sphere radius=0.09
- link panda_link4: geometry collision cylinder length=0.12 radius=0.09; collision sphere radius=0.09
- link panda_link5: geometry collision cylinder length=0.1 radius=0.09; collision cylinder length=0.14 radius=0.055
- link panda_link6: geometry collision cylinder length=0.08 radius=0.08; collision sphere radius=0.08
- link panda_link7: geometry collision cylinder length=0.14 radius=0.07; collision sphere radius=0.07

File: data/urdf/panda_hand.urdf (robot description, URDF)
Before this commit: robot panda_hand, 14 links, 13 joints
Links:
- link panda_hand: geometry collision cylinder length=0.1 radius=0.02; collision cylinder length=0.1 radius=0.04
- link panda_leftfinger: geometry visual mesh filename=file://@URDF_DESTINATION@/meshes/robot_arms/fr3/visual/fing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
- link panda_link0: geometry collision cylinder length=0.03 radius=0.09; collision sphere radius=0.09
- link panda_link1: geometry collision cylinder length=0.2830 radius=0.09; collision sphere radius=0.09
- link panda_link2: geometry collision cylinder length=0.12 radius=0.09; collision sphere radius=0.09
- link panda_link3: geometry collision cylinder length=0.15 radius=0.09; collision sphere radius=0.09
- link panda_link4: geometry collision cylinder length=0.12 radius=0.09; collision sphere radius=0.09
- link panda_link5: geometry collision cylinder length=0.1 radius=0.09; collision cylinder length=0.14 radius=0.055
- link panda_link6: geometry collision cylinder length=0.08 radius=0.08; collision sphere radius=0.08
- link panda_link7: geometry collision cylinder length=0.14 radius=0.07; collision sphere radius=0.07
- link panda_rightfinger: geometry visual mesh filename=file://@URDF_DESTINATION@/meshes/robot_arms/fr3/visual/fing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

File: data/urdf/panda_pump.urdf (robot description, URDF)
Before this commit: robot panda_pump, 12 links, 11 joints
Links:
- link panda_link0: geometry collision cylinder length=0.03 radius=0.09; collision sphere radius=0.09
- link panda_link1: geometry collision cylinder length=0.2830 radius=0.09; collision sphere radius=0.09
- link panda_link2: geometry collision cylinder length=0.12 radius=0.09; collision sphere radius=0.09
- link panda_link3: geometry collision cylinder length=0.15 radius=0.09; collision sphere radius=0.09
- link panda_link4: geometry collision cylinder length=0.12 radius=0.09; collision sphere radius=0.09
- link panda_link5: geometry collision cylinder length=0.1 radius=0.09; collision cylinder length=0.14 radius=0.055
- link panda_link6: geometry collision cylinder length=0.08 radius=0.08; collision sphere radius=0.08
- link panda_link7: geometry collision cylinder length=0.14 radius=0.07; collision sphere radius=0.07

File: data/xacro/hand.xacro (robot description, xacro)
@@ -20,5 +20,5 @@
       <visual>
         <geometry>
-          <mesh filename="package://franka_description/meshes/visual/hand.dae"/>
+          <mesh filename="package://franka_description/meshes/robot_ee/franka_hand_white/visual/hand.dae"/>
         </geometry>
       </visual>
@@ -63,5 +63,5 @@
       <visual>
         <geometry>
-          <mesh filename="package://franka_description/meshes/visual/finger.dae"/>
+          <mesh filename="package://franka_description/meshes/robot_ee/franka_hand_white/visual/finger.dae"/>
         </geometry>
       </visual>
@@ -71,5 +71,5 @@
         <origin xyz="0 0 0" rpy="0 0 ${pi}"/>
         <geometry>
-          <mesh filename="package://franka_description/meshes/visual/finger.dae"/>
+          <mesh filename="package://franka_description/meshes/robot_ee/franka_hand_white/visual/finger.dae"/>
         </geometry>
       </visual>

File: data/xacro/panda.xacro (robot description, xacro)
@@ -29,5 +29,5 @@
         <origin xyz="0 0 0" rpy="0 0 0"/>
         <geometry>
-          <mesh filename="package://${package_name}/meshes/visual/link0.dae"/>
+          <mesh filename="package://${package_name}/meshes/robot_arms/fr3/visual/link0.dae"/>
         </geometry>
         <material name="">
@@ -65,5 +65,5 @@
         <origin xyz="0 0 0" rpy="0 0 0"/>
         <geometry>
-          <mesh filename="package://${package_name}/meshes/visual/link1.dae"/>
+          <mesh filename="package://${package_name}/meshes/robot_arms/fr3/visual/link1.dae"/>
         </geometry>
         <material name="">
@@ -109,5 +109,5 @@
         <origin xyz="0 0 0" rpy="0 0 0"/>
         <geometry>
-          <mesh filename="package://${package_name}/meshes/visual/link2.dae"/>
+          <mesh filename="package://${package_name}/meshes/robot_arms/fr3/visual/link2.dae"/>
         </geometry>
         <material name="">
@@ -153,5 +153,5 @@
         <origin xyz="0 0 0" rpy="0 0 0"/>
         <geometry>
-          <mesh filename="package://${package_name}/meshes/visual/link3.dae"/>
+          <mesh filename="package://${package_name}/meshes/robot_arms/fr3/visual/link3.dae"/>
         </geometry>
         <material name="">
@@ -197,5 +197,5 @@
         <origin xyz="0 0 0" rpy="0 0 0"/>
         <geometry>
-          <mesh filename="package://${package_name}/meshes/visual/link4.dae"/>
+          <mesh filename="package://${package_name}/meshes/robot_arms/fr3/visual/link4.dae"/>
         </geometry>
         <material name="">
@@ -241,5 +241,5 @@
         <origin xyz="0 0 0" rpy="0 0 0"/>
         <geometry>
-          <mesh filename="package://${package_name}/meshes/visual/link5.dae"/>
+          <mesh filename="package://${package_name}/meshes/robot_arms/fr3/visual/link5.dae"/>
         </geometry>
         <material name="">
@@ -303,5 +303,5 @@
         <origin xyz="0 0 0" rpy="0 0 0"/>
         <geometry>
-          <mesh filename="package://${package_name}/meshes/visual/link6.dae"/>
+          <mesh filename="package://${package_name}/meshes/robot_arms/fr3/visual/link6.dae"/>
         </geometry>
         <material name="">
@@ -347,5 +347,5 @@
         <origin xyz="0 0 0" rpy="0 0 0"/>
         <geometry>
-          <mesh filename="package://${package_name}/meshes/visual/link7.dae"/>
+          <mesh filename="package://${package_name}/meshes/robot_arms/fr3/visual/link7.dae"/>
         </geometry>
         <material name="">
