Commit message: wip(tools)

File: data/urdf/panda_default.urdf (robot description, URDF)
Before this commit: robot panda_default, 11 links, 10 joints
Links:
- added link ball_link; visual sphere radius=0.005
Joints:
- added joint ball_joint: type fixed, parent panda_link8, child ball_link, origin xyz=-9.572068454947417e-05 0.00031346947529715616 0.07461399444599627 rpy=0.0 0.0 0.0

File: data/urdf/panda_hand.urdf (robot description, URDF)
Before this commit: robot panda_hand, 14 links, 13 joints
Links:
- removed link panda_hand
- removed link panda_leftfinger
- removed link panda_rightfinger
Joints:
- removed joint panda_finger_joint1
- removed joint panda_finger_joint2
- removed joint panda_hand_joint
