Commit message: wip: Install both fr1 and fr3 models

File: data/fr1/urdf/panda_default.in.urdf (robot description, URDF)
Before this commit: robot panda_default, 12 links, 11 joints
Links:
- removed link ball_link
- link panda_link0: geometry collision cylinder length=0.03 radius=0.09; collision sphere radius=0.09
- link panda_link1: geometry collision cylinder length=0.2830 radius=0.09; collision sphere radius=0.09
- link panda_link2: geometry collision cylinder length=0.12 radius=0.09; collision sphere radius=0.09
- link panda_link3: geometry collision cylinder length=0.15 radius=0.09; collision sphere radius=0.09
- link panda_link4: geometry collision cylinder length=0.12 radius=0.09; collision sphere radius=0.09
- link panda_link5: geometry collision cylinder length=0.1 radius=0.09; collision cylinder length=0.14 radius=0.055
- link panda_link6: geometry collision cylinder length=0.08 radius=0.08; collision sphere radius=0.08
- link panda_link7: geometry collision cylinder length=0.14 radius=0.07; collision sphere radius=0.07
Joints:
- removed joint ball_joint

File: data/fr1/urdf/panda_hand.urdf (robot description, URDF)
Before this commit: robot panda_hand, 11 links, 10 joints
Links:
- added link panda_hand, mass 0.73; collision cylinder length=0.1 radius=0.02; collision cylinder length=0.1 radius=0.04
- added link panda_leftfinger; visual mesh filename=file://@URDF_DESTINATION@/meshes/visual/finger.dae
- added link panda_rightfinger; visual mesh filename=file://@URDF_DESTINATION@/meshes/visual/finger.dae
Joints:
- added joint panda_finger_joint1: type prismatic, parent panda_hand, child panda_leftfinger, origin xyz=0 0 0.0584 rpy=0 0 0, axis 0 1 0, limit lower=0.0 upper=0.04 effort=20 velocity=0.2
- added joint panda_finger_joint2: type prismatic, parent panda_hand, child panda_rightfinger, origin xyz=0 0 0.0584 rpy=0 0 0, axis 0 -1 0, limit lower=0.0 upper=0.04 effort=20 velocity=0.2, mimic joint=panda_finger_joint1
- added joint panda_hand_joint: type fixed, parent panda_link8, child panda_hand, origin xyz=0 0 0 rpy=0 0 -0.7853981633974483
