Commit message: wip: Connect hand tool

File: data/tools/urdf/panda_hand.in.urdf (robot description, URDF)
Before this commit: robot panda_hand, 3 links, 3 joints
Links:
- added link panda_hand_connector
Joints:
- joint panda_hand_joint: parent panda_link8 -> panda_hand_connector

Commit message: wip: Connect pump, foot
How about devices in connected modules?

File: data/tools/urdf/panda_hand.in.urdf (robot description, URDF)
Before this commit: robot panda_hand, 4 links, 3 joints
Links:
- removed link panda_hand_connector
- added link tool_connector
Joints:
- joint panda_hand_joint: parent panda_hand_connector -> tool_connector
